File: RGB.kicad_sch (KiCad schematic)
At the start: 174 parts

Commit message: .
Connections:
- net RGB In: now reaches RGB1.4 (DIN)
Changed lines of the file:
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@@
+		)
+	)
+	(global_label "RGB In"
+		(shape input)
+		(at 393.7 22.86 0)
+		(fields_autoplaced yes)
+		(effects
+			(font
+				(size 1.27 1.27)
+			)
+			(justify left)
+		)
+		(property "Intersheetrefs" "${INTERSHEET_REFS}"
+			(at 403.2166 22.86 0)
+			(effects
+				(font
+					(size 1.27 1.27)
+				)
+				(justify left)
+				(hide yes)
+			)
 		)
 	)
